Commit message: Integrate RM-ECO65 as independent polishing-simulation project
- Replace Motoman hc10 with RM-ECO65 (rm_eco65), joint1-6, IK baselink->Link6
- Add rm_description urdf/xacro, 9 eco65 STL meshes, docker/compose + Dockerfile.custom
- Add toolpath/layout/IK analysis scripts and CN usage guides (docs/)
- part_scan.ply vertices shifted dx=-0.32 for eco65 layout
- Excludes runtime/ artifacts and nested src/ clone

File: urdf/ros2_control.xacro (robot description, xacro)
@@ -8,5 +8,5 @@
         </xacro:if>
       </hardware>
-      <joint name="${prefix}joint_1_s">
+      <joint name="${prefix}joint1">
         <command_interface name="position">
           <param name="min">${radians(-180)}</param>
@@ -21,5 +21,5 @@
         <state_interface name="velocity"/>
       </joint>
-      <joint name="${prefix}joint_2_l">
+      <joint name="${prefix}joint2">
         <command_interface name="position">
           <param name="min">${radians(-180)}</param>
@@ -34,5 +34,5 @@
         <state_interface name="velocity"/>
       </joint>
-      <joint name="${prefix}joint_3_u">
+      <joint name="${prefix}joint3">
         <command_interface name="position">
           <param name="min">${radians(-5)}</param>
@@ -45,9 +45,9 @@
         <command_interface name="acceleration"/>
         <state_interface name="position">
-          <param name="initial_value">${radians(90)}</param>
+          <param name="initial_value">0.0</param>
         </state_interface>
         <state_interface name="velocity" />
       </joint>
-      <joint name="${prefix}joint_4_r">
+      <joint name="${prefix}joint4">
         <command_interface name="position">
           <param name="min">${radians(-180)}</param>
@@ -62,5 +62,5 @@
         <state_interface name="velocity"/>
       </joint>
-      <joint name="${prefix}joint_5_b">
+      <joint name="${prefix}joint5">
         <command_interface name="position">
           <param name="min">${radians(-180)}</param>
@@ -75,5 +75,5 @@
         <state_interface name="velocity"/>
       </joint>
-      <joint name="${prefix}joint_6_t">
+      <joint name="${prefix}joint6">
         <command_interface name="position">
           <param name="min">${radians(-180)}</param>
@@ -86,5 +86,5 @@
         <command_interface name="acceleration"/>
         <state_interface name="position">
-          <param name="initial_value">0.785</param>
+          <param name="initial_value">0.0</param>
         </state_interface>
         <state_interface name="velocity"/>

File: urdf/workcell.xacro (robot description, xacro)
@@ -1,6 +1,7 @@
 <?xml version="1.0" ?>
-<robot name="motoman_hc10" xmlns:xacro="http://ros.org/wiki/xacro" xmlns:tesseract="https://github.com/tesseract-robotics/tesseract" tesseract:make_convex="true">
-  <xacro:include filename="$(find motoman_hc10_support)/urdf/hc10dt_macro.xacro" />
-  <xacro:motoman_hc10dt prefix=""/>
+<robot name="rm_eco65_workcell" xmlns:xacro="http://ros.org/wiki/xacro" xmlns:tesseract="https://github.com/tesseract-robotics/tesseract" tesseract:make_convex="true">
+  <!-- 直接引入本地的 eco65 URDF 文件 -->
+  <xacro:include filename="$(find snp_automate_2023)/urdf/rm_description/rm_eco65.urdf.xacro" />
+  <xacro:arg name="link6_type" default="Link6"/>
   <xacro:include filename="$(find snp_automate_2023)/urdf/ros2_control.xacro"/>
   <xacro:snp_ros2_control name="snp_ros2_control" prefix=""/>
@@ -61,5 +62,5 @@
   <joint name="table_to_base" type="fixed">
     <parent link="table"/>
-    <child link="base_link"/>
+    <child link="baselink"/>
     <origin xyz="-0.61 0 0.723" rpy="0 0 0"/>
   </joint>
@@ -143,5 +144,5 @@
   </link>
   <joint name="tool0_to_ee" type="fixed">
-    <parent link="tool0"/>
+    <parent link="Link6"/>
     <child link="ee"/>
     <origin rpy="0.0 0.0 ${radians(45)}"/>
@@ -156,5 +157,5 @@
   <link name="camera_frame"/>
   <joint name="tool0_to_camera" type="fixed">
-    <parent link="flange"/>
+    <parent link="Link6"/>
     <child link="camera_frame"/>
     <origin xyz="${camera_cal['camera_mount_to_camera_pos']['x']} ${camera_cal['camera_mount_to_camera_pos']['y']} ${camera_cal['camera_mount_to_camera_pos']['z']}"
@@ -175,9 +176,6 @@
   </link>
   <joint name="sand_tcp_joint" type="fixed">
-    <parent link="tool0"/>
-<!--    <origin xyz="-0.158 -0.158 0.123" rpy="0.0 ${radians(90)} ${radians(-135)}"/>-->
+    <parent link="Link6"/>
     <origin xyz="-0.149 ${-0.149 - 0.005} 0.083" rpy="0.0 ${radians(-90)} ${radians(-135)}"/>
-<!--    <parent link="ee"/>-->
-<!--    <origin xyz="${-0.186 - 0.038} 0.0 ${0.08325}" rpy="0.0 ${radians(90)} 0.0"/>-->
     <child link="sand_tcp"/>
   </joint>
